File: MOSH/MOSH.kicad_pcb (KiCad board)
At the start: 2 copper layers, 68.6 x 62.2 mm, 25 parts, among them J1 Power, J2 Digital/PWM, J3 Analog, J4 Digital/PWM, J5 Conn_01x08_Socket, J6 Conn_01x03_Pin, Q1 IRF540N, U1 LTC1050, U2 MCP41100

Commit message: j'ai fini de router, c'est pas opti mais ça existe
Routing:
- net ADC: track 68.7 -> 81.4 mm, vias 0 -> 1
Changed lines of the file:
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@@
         (effects (font (size 1 1) (thickness 0.15)))
     )
-    (fp_text value "Digital/PWM" (at 3.81 11.43 180) (layer "F.Fab")
-        (effects (font (size 1 1) (thickness 0.15)))
-    )
-    (fp_text user "${REFERENCE}" (at 3.81 0) (layer "F.Fab")
+    (fp_text value "Digital/PWM" (at 2.54 11.43 180) (layer "F.Fab")
+        (effects (font (size 1 1) (thickness 0.15)))
+    )
+    (fp_text user "${REFERENCE}" (at 2.54 0) (layer "F.Fab")
         (effects (font (size 1 1) (thickness 0.15)))
     )
@@
         (effects (font (size 1 1) (thickness 0.15)))
     )
-    (fp_text value "Digital/PWM" (at 3.81 8.89 180) (layer "F.Fab")
-        (effects (font (size 1 1) (thickness 0.15)))
-    )
-    (fp_text user "${REFERENCE}" (at 3.81 0) (layer "F.Fab")
+    (fp_text value "Digital/PWM" (at 2.54 8.89 180) (layer "F.Fab")
+        (effects (font (size 1 1) (thickness 0.15)))
+    )
+    (fp_text user "${REFERENCE}" (at 2.54 0) (layer "F.Fab")
         (effects (font (size 1 1) (thickness 0.15)))
     )
@@
     (property "ki_keywords" "R res resistor")
     (attr through_hole)
-    (fp_text reference "R4" (at 42.32 14.76 90) (layer "F.SilkS")
+    (fp_text reference "R4" (at 6.35 0 90) (layer "F.SilkS")
         (effects (font (size 1 1) (thickness 0.15)))
     )
@@
         (effects (font (size 1 1) (thickness 0.15)))
     )
-    (fp_text user "${REFERENCE}" (at 7.62 -50.72) (layer "F.Fab")
+    (fp_text user "${REFERENCE}" (at 5.08 3.81) (layer "F.Fab")
         (effects (font (size 1 1) (thickness 0.15)))
     )
@@
   (segment (start 133.02 56.82) (end 136.576 53.264) (width 0.8) (layer "B.Cu") (net 16))
   (segment (start 130.48 56.82) (end 133.02 56.82) (width 0.8) (layer "B.Cu") (net 16))
+  (segment (start 150.8 105.08) (end 150.8 97.46) (width 0.8) (layer "F.Cu") (net 17))
+  (via (at 150.8 105.08) (size 1.5) (drill 0.8) (layers "F.Cu" "B.Cu") (net 17))
+  (segment (start 110.324214 93.485786) (end 111.43 94.591572) (width 0.8) (layer "B.Cu") (net 17))
   (segment (start 103.81 77.14) (end 101.81 79.14) (width 0.8) (layer "B.Cu") (net 17))
-  (segment (start 111.64 101.48) (end 113.97 103.81) (width 0.8) (layer "B.Cu") (net 17))
-  (segment (start 108.89 89.88) (end 111.64 92.63) (width 0.8) (layer "B.Cu") (net 17))
-  (segment (start 111.64 92.63) (end 111.64 101.48) (width 0.8) (layer "B.Cu") (net 17))
+  (segment (start 108.89 89.88) (end 108.89 92.051572) (width 0.8) (layer "B.Cu") (net 17))
+  (segment (start 112.7 103.81) (end 130.48 103.81) (width 0.8) (layer "B.Cu") (net 17))
+  (segment (start 131.75 105.08) (end 150.8 105.08) (width 0.8) (layer "B.Cu") (net 17))
+  (segment (start 111.43 102.54) (end 112.7 103.81) (width 0.8) (layer "B.Cu") (net 17))
   (segment (start 101.81 88.128428) (end 103.561572 89.88) (width 0.8) (layer "B.Cu") (net 17))
   (segment (start 103.561572 89.88) (end 108.89 89.88) (width 0.8) (layer "B.Cu") (net 17))
+  (segment (start 130.48 103.81) (end 131.75 105.08) (width 0.8) (layer "B.Cu") (net 17))
   (segment (start 101.81 79.14) (end 101.81 88.128428) (width 0.8) (layer "B.Cu") (net 17))
-  (segment (start 113.97 103.81) (end 146.99 103.81) (width 0.8) (layer "B.Cu") (net 17))
+  (segment (start 111.43 94.591572) (end 111.43 102.54) (width 0.8) (layer "B.Cu") (net 17))
+  (segment (start 108.89 92.051572) (end 110.324214 93.485786) (width 0.8) (layer "B.Cu") (net 17))
   (segment (start 150.8 83.49) (end 148.26 80.95) (width 0.8) (layer "B.Cu") (net 19))
   (segment (start 157.15 86.03) (end 154.61 83.49) (width 0.8) (layer "B.Cu") (net 19))
